Commit message: Updated goal_track to send goals and added nav2 testing modified
vlm_vision:
Fixed bugs with goal_track node
Allowed goal_track to send goals from base_link to goal frame
implemented goal thresholding

unitree:
Added frame for mounted camera
Added transform from map to odom and base_link for testing mode

File: unitree/go2_description/xacro/robot.xacro (robot description, xacro)
@@ -81,4 +81,11 @@
         </collision>
     </link>
+    <joint name="mounted_camera" type="fixed">
+        <parent link="trunk"/>
+        <child link="mounted_camera"/>
+        <origin rpy="0 1.5708 0" xyz="0.29515 -0.00003 0.06"/>
+    </joint>
+    <link name="mounted_camera">
+    </link>
     <joint name="front_camera_joint" type="fixed">
         <parent link="trunk"/>

Commit message: Added service to goal_track to send a goal pose Fixed xacro file for correct camera orientation

File: unitree/go2_description/xacro/robot.xacro (robot description, xacro)
@@ -84,5 +84,5 @@
         <parent link="trunk"/>
         <child link="mounted_camera"/>
-        <origin rpy="0 1.5708 0" xyz="0.29515 -0.00003 0.06"/>
+        <origin rpy="3.1416 -1.5708 0" xyz="0.29515 -0.00003 0.06"/>
     </joint>
     <link name="mounted_camera">

Commit message: Implemented rtabmap.launch.py to launch rtab slam mapping and the rtab visualizer Created rtab_params to store params for RGBD and lidar sensor fusion mapping (mode 2) Updated nav2.launch and nav2 params to work with rolling cost map Updated nav rviz file to show joint publisher, map, and point clouds Updated robot.xacro to publish lidar tf frame

File: unitree/go2_description/xacro/robot.xacro (robot description, xacro)
@@ -56,4 +56,11 @@
         </inertial>
     </link>
+    <joint name="lidar_joint" type="fixed">
+        <parent link="trunk"/>
+        <child link="utlidar_lidar"/>
+        <origin rpy="0 -0.2 0" xyz="0.29515 -0.00003 -0.06597"/>
+    </joint>
+    <link name="utlidar_lidar">
+    </link>
     <joint name="imu_joint" type="fixed">
         <parent link="trunk"/>
@@ -81,10 +88,10 @@
         </collision>
     </link>
-    <joint name="mounted_camera" type="fixed">
+    <joint name="camera_joint" type="fixed">
         <parent link="trunk"/>
-        <child link="mounted_camera"/>
+        <child link="camera_link"/>
         <origin rpy="3.1416 -1.5708 0" xyz="0.29515 -0.00003 0.06"/>
     </joint>
-    <link name="mounted_camera">
+    <link name="camera_link">
     </link>
     <joint name="front_camera_joint" type="fixed">

Commit message: Debugged rtab params problems changed camera link to not project upwards added camera vision link

File: unitree/go2_description/xacro/robot.xacro (robot description, xacro)
@@ -91,7 +91,17 @@
         <parent link="trunk"/>
         <child link="camera_link"/>
+        <origin rpy="0 0 0" xyz="0.29515 -0.00003 0.06"/>
+    </joint>
+    <link name="camera_link">
+    </link>
+    <!-- Separate frame used by the vision goal pipeline.
+         Keeps the original rotation so that z_m (depth) maps to the forward
+         direction expected by goal_track's TF broadcast. -->
+    <joint name="camera_vision_joint" type="fixed">
+        <parent link="trunk"/>
+        <child link="camera_vision_link"/>
         <origin rpy="3.1416 -1.5708 0" xyz="0.29515 -0.00003 0.06"/>
     </joint>
-    <link name="camera_link">
+    <link name="camera_vision_link">
     </link>
     <joint name="front_camera_joint" type="fixed">
